File: crates/pcb-layout/tests/resources/zones/module/layout.kicad_pcb (KiCad board)
At the start: 2 copper layers, 4 parts

Commit message: simpler zone test
Parts:
- removed R3, R4: 1k, R_0603_1608Metric:R_0603_1608Metric
- R1: moved to F.Cu
- moved R1 2.31 mm to (147.0, 104.0)
- moved R2 1.52 mm to (150.0, 104.0)
Routing:
- removed copper zone on B.Cu, net P2
