File: crates/pcb-layout/tests/resources/complex/module/layout.kicad_pcb (KiCad board)
At the start: 2 copper layers, 4 parts

Commit message: sync vias and track
Routing:
- net P1: track 0.00 -> 17.8 mm, vias 0 -> 2
- net P2: track 0.00 -> 5.96 mm, vias 0 -> 2
