File: stdlib/test/layout/test_BoardConfig/layout.kicad_pcb (KiCad board)
At the start: 8 copper layers, 0 parts

Commit message: Update stdlib test layout files to KiCad 10
Other:
- copper layers 8 -> 4
Changed lines of the file:
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@@
 (kicad_pcb
-	(version 20241229)
+	(version 20260206)
 	(generator "pcbnew")
-	(generator_version "9.0")
+	(generator_version "10.0")
 	(general
-		(thickness 1.6)
+		(thickness 1.6062)
 		(legacy_teardrops no)
 	)
@@
 		(4 "In1.Cu" power)
 		(6 "In2.Cu" power)
-		(8 "In3.Cu" mixed)
-		(10 "In4.Cu" power)
-		(12 "In5.Cu" mixed)
-		(14 "In6.Cu" power)
 		(2 "B.Cu" mixed)
 		(9 "F.Adhes" user "F.Adhesive")
@@
 	)
 	(setup
-		(stackup
-  (layer
-    "F.SilkS"
-    (type "Top Silk Screen")
-    (color "White")
-  )
-  (layer
-    "F.Paste"
-    (type "Top Solder Paste")
-  )
-  (layer
-    "F.Mask"
-    (type "Top Solder Mask")
-    (color "Black")
-    (thickness 0.01)
-  )
-  (layer
-    "F.Cu"
-    (type "copper")
-    (thickness 0.035)
-  )
-  (layer
-    "dielectric 1"
-    (type "prepreg")
-    (thickness 0.1164)
-    (material "2116")
-    (epsilon_r 4.16)
-    (loss_tangent 0.025)
-  )
-  (layer
-    "In1.Cu"
-    (type "copper")
-    (thickness 0.0152)
-  )
-  (layer
-    "dielectric 2"
-    (type "core")
-    (thickness 0.3)
-    (material "FR4-Core")
-    (epsilon_r 4.6)
-    (loss_tangent 0.025)
-  )
-  (layer
-    "In2.Cu"
-    (type "copper")
-    (thickness 0.0152)
-  )
-  (layer
-    "dielectric 3"
-    (type "prepreg")
-    (thickness 0.0764)
-    (material "1080")
-    (epsilon_r 3.91)
-    (loss_tangent 0.025)
-    addsublayer
-    (type "prepreg")
-    (thickness 0.0764)
-    (material "1080")
-    (epsilon_r 3.91)
-    (loss_tangent 0.025)
-  )
-  (layer
-    "In3.Cu"
-    (type "copper")
-    (thickness 0.0152)
-  )
-  (layer
-    "dielectric 4"
-    (type "core")
-    (thickness 0.3)
-    (material "FR4-Core")
-    (epsilon_r 4.6)
-    (loss_tangent 0.025)
-  )
-  (layer
-    "In4.Cu"
-    (type "copper")
-    (thickness 0.0152)
-  )
-  (layer
-    "dielectric 5"
-    (type "prepreg")
-    (thickness 0.0764)
-    (material "1080")
-    (epsilon_r 3.91)
-    (loss_tangent 0.025)
-    addsublayer
-    (type "prepreg")
-    (thickness 0.0764)
-    (material "1080")
-    (epsilon_r 3.91)
-    (loss_tangent 0.025)
-  )
-  (layer
-    "In5.Cu"
-    (type "copper")
-    (thickness 0.0152)
-  )
-  (layer
-    "dielectric 6"
-    (type "core")
-    (thickness 0.3)
-    (material "FR4-Core")
-    (epsilon_r 4.6)
-    (loss_tangent 0.025)
-  )
-  (layer
-    "In6.Cu"
-    (type "copper")
-    (thickness 0.0152)
-  )
-  (layer
-    "dielectric 7"
-    (type "prepreg")
-    (thickness 0.1164)
-    (material "2116")
-    (epsilon_r 4.16)
-    (loss_tangent 0.025)
-  )
-  (layer
-    "B.Cu"
-    (type "copper")
-    (thickness 0.035)
-  )
-  (layer
-    "B.Mask"
-    (type "Bottom Solder Mask")
-    (color "Black")
-    (thickness 0.01)
-  )
-  (layer
-    "B.Paste"
-    (type "Bottom Solder Paste")
-  )
-  (layer
-    "B.SilkS"
-    (type "Bottom Silk Screen")
-    (color "White")
-  )
-  (copper_finish "ENIG")
-  (dielectric_constraints no)
-)
 		(pad_to_mask_clearance 0)
 		(allow_soldermask_bridges_in_footprints no)
-		(tenting front back)
+		(tenting
+			(front yes)
+			(back yes)
+		)
+		(covering
+			(front no)
+			(back no)
+		)
+		(plugging
+			(front no)
+			(back no)
+		)
+		(capping no)
+		(filling no)
 		(pcbplotparams
 			(layerselection 0x00000000_00000000_55555555_5755f5ff)
@@
 			(usegerberadvancedattributes yes)
 			(creategerberjobfile yes)
-			(dashed_line_dash_ratio 12.000000)
-			(dashed_line_gap_ratio 3.000000)
+			(dashed_line_dash_ratio 12)
+			(dashed_line_gap_ratio 3)
 			(svgprecision 4)
 			(plotframeref no)
 			(mode 1)
 			(useauxorigin no)
-			(hpglpennumber 1)
-			(hpglpenspeed 20)
-			(hpglpendiameter 15.000000)
 			(pdf_front_fp_property_popups yes)
 			(pdf_back_fp_property_popups yes)
@@
 			(outputdirectory "")
 		)
+		(stackup
+			(layer "F.SilkS"
+				(type "Top Silk Screen")
+				(color "White")
+			)
+			(layer "F.Paste"
+				(type "Top Solder Paste")
+			)
+			(layer "F.Mask"
+				(type "Top Solder Mask")
+				(color "Black")
+				(thickness 0.01)
+			)
+			(layer "F.Cu"
+				(type "copper")
+				(thickness 0.035)
+			)
+			(layer "dielectric 1"
+				(type "prepreg")
+				(thickness 0.2104)
+				(material "Prepreg")
+				(epsilon_r 4.4)
+				(loss_tangent 0.025)
+			)
+			(layer "In1.Cu"
+				(type "copper")
+				(thickness 0.0152)
+			)
+			(layer "dielectric 2"
+				(type "core")
+				(thickness 1.065)
+				(material "FR4-Core")
+				(epsilon_r 4.6)
+				(loss_tangent 0.025)
+			)
+			(layer "In2.Cu"
+				(type "copper")
+				(thickness 0.0152)
+			)
+			(layer "dielectric 3"
+				(type "prepreg")
+				(thickness 0.2104)
+				(material "Prepreg")
+				(epsilon_r 4.4)
+				(loss_tangent 0.025)
+			)
+			(layer "B.Cu"
+				(type "copper")
+				(thickness 0.035)
+			)
+			(layer "B.Mask"
+				(type "Bottom Solder Mask")
+				(color "Black")
+				(thickness 0.01)
+			)
+			(layer "B.Paste"
+				(type "Bottom Solder Paste")
+			)
+			(layer "B.SilkS"
+				(type "Bottom Silk Screen")
+				(color "White")
+			)
+			(copper_finish "ENIG")
+			(dielectric_constraints no)
+		)
 	)
-	(net 0 "")
 	(embedded_fonts no)
 )
