File: crates/pcb-kicad-sch/test-data/kicad-10/resaved-child-sheet.kicad_sch (KiCad schematic)
At the start: 2 parts

Commit message: ENG-3825 Fix review findings since v0.4.74 and simplify the changed code
Fix title_block order in written schematics, pcb migrate with a positional
Board() name, the DFM report file mode, a lingering legacy Val field, and
exclude_from_sim in pcb import and in text items. Share STEP and glTF
geometry helpers, build the DFM scene only for a database, remove dead
schematic identity code, and parse the property private flag in one place.
Update the Unreleased changelog and stale docs.
Other:
- title: (none) -> Fixture
Changed lines of the file:
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@@
 	(generator_version "10.0")
 	(paper "A4")
+	(title_block
+		(title "Fixture")
+		(rev "A")
+	)
 	(wire
 		(pts
